File: OPD-Computer-One-Disk-Interface.kicad_pcb (KiCad board)
At the start: 2 copper layers, 82 x 76 mm, 22 parts, among them IC1 WD1772, IC2 27C128, IC3 74LS245, IC4 74LS175, IC5 GAL16V8, IC6 74LS06, IC7 74LS06, J1 Host Connector, J2 Floppy Connector, X1 8MHz Crystal Oscillator

Commit message: Fixed typo in copyright date on rear silkscreen.
Other:
- board text added: "OPD Computer One Floppy Interface Recreation ©2024 Stephen Usher"
- board text removed: "OPD Computer One Floppy Interface Recreation ©2014 Stephen Usher"
Changed lines of the file:
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@@
 		)
 	)
-	(gr_text "OPD Computer One\nFloppy Interface Recreation\n©2014 Stephen Usher"
+	(gr_text "OPD Computer One\nFloppy Interface Recreation\n©2024 Stephen Usher"
 		(at 106.1 100.7 270)
 		(layer "B.SilkS")
